File: sensor-stack/PIC SENSOR-BOARD.sch (EAGLE design)
At the start: 27 parts

Commit message: Added Sensor Board
Parts:
- removed LED10, LED11, LED12, LED13, LED14, LED15, LED16: (no value), eagle-ltspice:LED_E
- removed XB1: XBEE, maxstream:XBEE
- added C1, C2: (no value), rcl:C-USC0805
- added D1: RGB, SparkFun-LED:LED-RGBPLCC-6
- added H5, H6: MOUNT-PAD-ROUND3.3, holes:MOUNT-PAD-ROUND3.3
- added JP3, JP5: (no value), pinhead:PINHD-1X2
- added JP4: (no value), adafruit:PINHD-2X20
- added LED1, LED2, LED3, LED4, LED5, LED6, LED7, LED8: (no value), led:LEDSML0603
- added R17, R18, R22, R23, R24: (no value), rcl:R-US_R0805
- added R19, R20, R21, R25, R26, R5, R6, R7, R8: (no value), rcl:R-US_M0805
- added S1, S2: MOMENTARY-SWITCH-SPST-PTH-6.0MM, SparkFun-Switches:MOMENTARY-SWITCH-SPST-PTH-6.0MM
- added SJ1, SJ10, SJ11, SJ12, SJ13, SJ14, SJ15, SJ16, SJ17, SJ18, SJ19, SJ2, SJ20, SJ21, SJ22, SJ23, SJ24, SJ25, SJ3, SJ4, SJ5, SJ6, SJ7, SJ8, SJ9: (no value), jumper:SJ
- added SW1: DIP-06, SparkFun-Switches:DIP-06
- added TM1: (no value), adafruit:TRIMPOT3386
- added U$1: ACS723, SparkFun-Sensors:ACS723
- added U$2: TEMP-HUM-SENSOR-DHT11, diy-modules:TEMP-HUM-SENSOR-DHT11
- added U1, U2: TMP36GSZ, ADI-Phase-2:TMP36GSZ
- JP1: device pinhead:PINHD-1X20 -> pinhead:PINHD-1X2
- JP2: device pinhead:PINHD-1X20 -> adafruit:PINHD-2X20
- LED9: device eagle-ltspice:LED_E -> led:LEDCHIPLED_0603
- R1: value (none) -> PHOTOCELLPTH; device rcl:R-US_R0805 -> SparkFun-Sensors:PHOTOCELLPTH
- R13, R14, R15, R16: device rcl:R-US_M0805 -> rcl:R-US_R0805
- R2, R4: device rcl:R-US_R0805 -> rcl:R-US_M0805
- R3: value (none) -> 5K; device rcl:R-US_R0805 -> rcl:R-US_M0805
Connections:
- removed net N$10: LED10.A
- removed net N$11: LED11.A
- removed net N$12: LED12.A
- removed net N$13: LED13.A
- removed net N$14: LED14.A
- removed net N$15: LED15.A
- removed net N$16: LED16.A
- removed net N$17: LED9.C, R9.2
- removed net N$18: LED10.C, R10.2
- removed net N$19: LED11.C, R11.2
- removed net N$2: R3.2, R4.2, XB1.DIN/!CONFIG
- removed net N$20: LED12.C, R12.2
- removed net N$21: LED13.C, R13.2
- removed net N$22: LED14.C, R14.2
- removed net N$23: LED15.C, R15.2
- removed net N$24: LED16.C, R16.2
- removed net N$3: R1.2, R2.2, XB1.DOUT
- removed net N$9: LED9.A
- removed net RA0: JP1.2
- removed net RA1: JP1.3
- removed net RA2: JP1.4
- removed net RA3: JP1.5
- removed net RA4: JP1.6
- removed net RA5: JP1.7
- removed net RA6: JP1.14
- removed net RA7: JP1.13
- removed net RB0: JP2.8
- removed net RB1: JP2.7
- removed net RB2: JP2.6
- removed net RB3: JP2.5
- removed net RB4: JP2.4
- removed net RB5: JP2.3
- removed net RD0: JP1.19
- removed net RD1: JP1.20
- removed net RD2: JP2.20
- removed net RD3: JP2.19
- removed net RD4: JP2.14
- removed net RD5: JP2.13
- removed net RD6: JP2.12
- removed net RD7: JP2.11
- removed net RE0: JP1.8
- removed net RE1: JP1.9
- removed net RE2: JP1.10
- new net BLUE+: D1.BLU-A, SJ16.1
- new net BLUE-: D1.BLU-C, R24.1
- new net BLUE_ON: JP2.19, JP2.20, SJ16.2
- new net CAP2_NEG: C1.2, R19.1, SJ14.1
- new net CAP_NEG: C2.2, R21.1, SJ15.1
- new net CURRENT_LINE: SJ2.1, U$1.VIOUT
- new net CURRENT_OUT: JP4.21, JP4.22, SJ2.2
- new net DIP1_LINE: R13.2, SJ25.1, SW1.1
- new net DIP1_OUT: JP4.15, JP4.16, SJ25.2
- new net DIP2_LINE: R14.2, SJ24.1, SW1.2
- new net DIP2_OUT: JP4.13, JP4.14, SJ24.2
- new net DIP3_LINE: R15.2, SJ23.1, SW1.3
- new net DIP3_OUT: JP4.11, JP4.12, SJ23.2
- new net DIP4_LINE: R16.2, SJ22.1, SW1.4
- new net DIP4_OUT: JP4.10, JP4.9, SJ22.2
- new net DIP5_LINE: R17.2, SJ21.1, SW1.5
- new net DIP5_OUT: JP4.7, JP4.8, SJ21.2
- new net DIP6_LINE: R18.2, SJ20.1, SW1.6
- new net DIP6_OUT: JP4.5, JP4.6, SJ20.2
- new net GREEN+: D1.GRN-A, SJ17.1
- new net GREEN-: D1.GRN-C, R23.1
- new net GREEN_ON: JP2.17, JP2.18, SJ17.2
- new net HUM_DATA: R3.1, SJ5.2, U$2.DAT
- new net HUM_OUT: JP4.25, JP4.26, SJ5.1
- new net IP+: H5.MOUNT, JP3.2, U$1.IP+@1, U$1.IP+@2
- new net IP-: H6.MOUNT, JP3.1, U$1.IP-@1, U$1.IP-@2
- new net L1+: LED1.A, SJ6.1
- new net L1-: LED1.C, R5.2
- new net L2+: LED2.A, SJ7.1
- new net L2-: LED2.C, R6.2
- new net L3+: LED3.A, SJ8.1
- new net L3-: LED3.C, R7.2
- new net L4+: LED4.A, SJ9.1
- new net L4-: LED4.C, R8.2
- new net L5+: LED5.A, SJ10.1
- new net L5-: LED5.C, R9.2
- new net L6+: LED6.A, SJ11.1
- new net L6-: LED6.C, R10.2
- new net L7+: LED7.A, SJ12.1
- new net L7-: LED7.C, R11.2
- new net L8+: LED8.A, SJ13.1
- new net L8-: LED8.C, R12.2
- new net LED1_ON: JP2.3, JP2.4, SJ6.2
- new net LED2_ON: JP2.5, JP2.6, SJ7.2
- new net LED3_ON: JP2.7, JP2.8, SJ8.2
- new net LED4_ON: JP2.10, JP2.9, SJ9.2
- new net LED5_ON: JP2.11, JP2.12, SJ10.2
- new net LED6_ON: JP2.13, JP2.14, SJ11.2
- new net LED7_ON: JP2.27, JP2.28, SJ12.2
- new net LED8_ON: JP2.25, JP2.26, SJ13.2
- new net LIGHT_LINE: R1.P$1, R2.1, SJ1.1
- new net LIGHT_OUT: JP4.27, JP4.28, SJ1.2
- new net POWER-: LED9.C, R25.1
- new net RED+: D1.RED-A, SJ18.1
- new net RED-: D1.RED-C, R22.1
- new net RED_ON: JP2.15, JP2.16, SJ18.2
- new net SWITCH1_OUT: JP2.37, JP2.38, SJ15.2
- new net SWITCH2_OUT: JP2.39, JP2.40, SJ14.2
- new net SW_NEG: R20.2, R21.2, S2.1
- new net SW_NEG2: R19.2, R4.2, S1.1
- new net T1_LINE: SJ4.1, U1.VOUT
- new net T2_LINE: SJ3.1, U2.VOUT
- new net TEMP1_OUT: JP4.39, JP4.40, SJ4.2
- new net TEMP2_OUT: JP4.37, JP4.38, SJ3.2
- new net TRIM: R26.2, TM1.E
- new net TRIM_JUMP: SJ19.2, TM1.S
- new net TRIM_OUT: JP4.23, JP4.24, SJ19.1
- net GND: now also JP1.1, JP2.23, JP2.24, JP4.19, JP4.20, JP5.1, R1.P$2, R17.1, R18.1, R20.1, R22.2, R23.2, R24.2, R25.2, R26.1, R4.1, R5.1, R6.1, R7.1, R8.1, U$1.BW_SEL, U$1.GND, U$2.GND, U1.GND, U2.GND; no longer JP1.12, JP2.10, XB1.GND
- net MCLR: now also JP2.1, JP2.2; no longer JP1.1
- net RB6/PGC: now also JP4.3, JP4.4; no longer JP2.2
- net RB7/PGD: now also JP4.1, JP4.2; no longer JP2.1
- net RC0: now also JP2.29, JP2.30; no longer JP1.15
- net RC1: now also JP2.31, JP2.32; no longer JP1.16
- net RC2: now also JP2.33, JP2.34; no longer JP1.17
- net RC3: now also JP2.35, JP2.36; no longer JP1.18
- net RC4: now also JP4.35, JP4.36; no longer JP2.18
- net RC5: now also JP4.33, JP4.34; no longer JP2.17
- net RC6: now also JP4.31, JP4.32; no longer JP2.16
- net RC7: now also JP4.29, JP4.30; no longer JP2.15
- net VDD: now also C1.1, C2.1, JP1.2, JP2.21, JP2.22, JP4.17, JP4.18, JP5.2, LED9.A, R2.2, R3.2, S1.2, S2.2, SW1.10, SW1.11, SW1.12, SW1.7, SW1.8, SW1.9, TM1.A, U$1.VCC, U$2.VDD, U1.+VS, U1.SHUTDOWN*, U2.+VS, U2.SHUTDOWN*; no longer JP1.11, JP2.9, XB1.VCC
Other:
- note added: "Board Voltage"
- note added: "Board with sensors that goes with the PIC18F45K40 breakout board. It also has programmable lights, analog devices, and actuators that can be used."
- note added: "Current Sensor"
- note added: "DIP SWITCHES"
- note added: "Debounced Momentary Switches"
- note added: "Enviromental Sensors"
- note added: "Humidity Sensor"
- note added: "Misc. Analog Sensors"
- note added: "Photoresistive Light Sensor"
- note added: "Power Indicator"
- note added: "RGB LED"
- note added: "Temperature Sensor 1"
- note added: "Temperature Sensor 2"
- note added: "Trimpot"
- note removed: "A user friendly breakout board for the PIC18F45K20 and similar chipset. Has onboard USB 5v to 3.3V at 1A."
